Commit message: Add launch file for autocar_ros and update URDF with camera integration

File: src/autocar_ros/urdf/autocar_ros.xacro (robot description, xacro)
@@ -1,4 +1,4 @@
 <?xml version="1.0"?>
-<robot name="follower_vehicle" xmlns:xacro="http://ros.org/wiki/xacro">
+<robot name="autocar_ros" xmlns:xacro="http://ros.org/wiki/xacro">
   <xacro:property name="r" value="0.3"/>
   <xacro:property name="w" value="0.25"/>
@@ -26,5 +26,5 @@
     </collision>
     <inertial>
-      <mass value="5.0"/>
+      <mass value="500.0"/>
       <inertia ixx="0.5" ixy="0" ixz="0" iyy="0.5" iyz="0" izz="0.5"/>
     </inertial>
@@ -66,27 +66,4 @@
   <xacro:wheel name="front_wheel_right" x="1.25" y="0.8" mu="5"/>
   <xacro:wheel name="front_wheel_left"  x="1.25" y="-0.8" mu="5"/>
-  <!-- Depth Camera Link -->
-  <link name="depth_camera_link">
-    <visual>
-      <geometry>
-        <box size="0.1 0.1 0.1"/>
-      </geometry>
-    </visual>
-    <collision>
-      <geometry>
-        <box size="0.1 0.1 0.1"/>
-      </geometry>
-    </collision>
-    <inertial>
-      <mass value="0.1"/>
-      <inertia ixx="0.000166667" ixy="0" ixz="0" iyy="0.000166667" iyz="0" izz="0.000166667"/>
-    </inertial>
-  </link>
-  <!-- Camera Joint (Fixed) -->
-  <joint name="chassis_depth_camera_fixed" type="fixed">
-    <parent link="chassis"/>
-    <child link="depth_camera_link"/>
-    <origin rpy="0 0 0" xyz="-0.1 0 1.25"/>
-  </joint>
   <!-- Differential Drive Plugin -->
   <gazebo>
@@ -105,29 +82,6 @@
     </plugin>
   </gazebo>
-  <gazebo reference="depth_camera_link">
-    <material>Gazebo/Black</material>
-    <sensor name="depth_camera" type="depth">
-      <update_rate>30.0</update_rate>
-      <camera>
-        <horizontal_fov>1.047</horizontal_fov>
-        <image>
-          <width>320</width>
-          <height>240</height>
-          <format>R8G8B8</format>
-        </image>
-        <clip>
-          <near>0.1</near>
-          <far>100</far>
-        </clip>
-      </camera>
-      <plugin name="depth_camera_controller" filename="libgazebo_ros_camera.so">
-        <alwaysOn>true</alwaysOn>
-        <updateRate>30.0</updateRate>
-        <cameraName>depth_camera</cameraName>
-        <imageTopicName>depth/image_raw</imageTopicName>
-        <cameraInfoTopicName>depth/camera_info</cameraInfoTopicName>
-        <frameName>depth_camera_link</frameName>
-      </plugin>
-    </sensor>
-  </gazebo>
+  <xacro:include filename="$(find autocar_ros)/urdf/sensors/simple_camera.xacro"/>
+  <xacro:simple_camera parent_link="chassis" name="camera_front"
+                      xyz="0.06 0 1.15" rpy="0 0 0"/>
 </robot>
